Commit message: Add files via upload

File: crx10ial.urdf (robot description, URDF)
Before this commit: robot fanuc_crx10ial, 9 links, 8 joints
Links:
- link base_link: mass 4.0 -> None
- link forearm_link: mass 2.275 -> None
- link shoulder_link: mass 3.7 -> None
- link upper_arm_link: mass 8.393 -> None
- link wrist_1_link: mass 1.219 -> None
- link wrist_2_link: mass 1.219 -> None
- link wrist_3_link: mass 0.1879 -> None
